File: LED_Torch/LED_Torch.kicad_pcb (KiCad board)
At the start: 2 copper layers, 4 parts, among them SW1 SW_DIP_x01

Commit message: LED Torch
Parts:
- moved D1 29.2 mm to (141.0, 70.0), turned to -90 degrees
- moved R1 21.0 mm to (117.2, 69.0)
- moved SW1 14.5 mm to (100.8, 75.8), turned to 90 degrees
- moved BT1 12.0 mm to (81.5, 70.0)
Routing:
- net Net-(BT1--): track 0.00 -> 68.3 mm
- net Net-(BT1-+): track 0.00 -> 33.1 mm
- net Net-(R1-Pad1): track 0.00 -> 18.5 mm
- net Net-(D1-A): track 0.00 -> 18.4 mm
Other:
- board outline added: 85.7 x 39.5 mm
