File: LED_Torch/LED_Torch.kicad_pcb (KiCad board)
At the start: 2 copper layers, 43.8 x 18.3 mm, 4 parts, among them SW1 SW_DIP_x01

Commit message: Traffic light
Other:
- board size 43.8 x 18.3 mm -> 80.5 x 46.2 mm
Changed lines of the file:
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@@
 		(tags "tact sw push 6mm")
 		(property "Reference" "SW1"
-			(at 3.25 -2 360)
+			(at 3.25 -2 0)
 			(layer "F.SilkS")
 			(effects
@@
 		)
 		(property "Value" "SW_DIP_x01"
-			(at 3.75 6.7 360)
+			(at 3.75 6.7 0)
 			(layer "F.Fab")
 			(effects
@@
 		)
 		(fp_text user "${REFERENCE}"
-			(at 3.25 2.25 360)
+			(at 3.25 2.25 0)
 			(layer "F.Fab")
 			(effects
@@
 		(tags "Keystone type 1058 coin cell retainer")
 		(property "Reference" "BT1"
-			(at 0 7.62 360)
+			(at 0 7.62 0)
 			(layer "F.SilkS")
 			(effects
@@
 		)
 		(property "Value" "Battery_Cell"
-			(at 0 -9.398 360)
+			(at 0 -9.398 0)
 			(layer "F.Fab")
 			(effects
@@
 		)
 		(fp_text user "${REFERENCE}"
-			(at 0 0 360)
+			(at 0 0 0)
 			(layer "F.Fab")
 			(effects
@@
 	)
 	(gr_arc
-		(start 51.000001 67)
-		(mid 70.527065 49.073744)
-		(end 94.799748 59.727088)
+		(start 96.423753 81.179863)
+		(mid 69.182743 93.509728)
+		(end 49.5 71)
 		(stroke
 			(width 0.05)
+			(type default)
+		)
+		(layer "Edge.Cuts")
+	)
+	(gr_line
+		(start 130 81.5)
+		(end 96.423753 81.179863)
+		(stroke
+			(width 0.05)
+			(type default)
+		)
+		(layer "Edge.Cuts")
+	)
+	(gr_arc
+		(start 49.5 71)
+		(mid 69.182743 48.490272)
+		(end 96.423753 60.820137)
+		(stroke
+			(width 0.05)
+			(type default)
+		)
+		(layer "Edge.Cuts")
+	)
+	(gr_line
+		(start 130 61)
+		(end 130 81.5)
+		(stroke
+			(width 0.05)
+			(type default)
+		)
+		(layer "Edge.Cuts")
+	)
+	(gr_line
+		(start 96.423753 60.820137)
+		(end 130 61)
+		(stroke
+			(width 0.05)

Commit message: IR Sensor
Parts:
- BT1: value Battery_Cell -> BH32T-C-G; footprint Battery:BatteryHolder_Keystone_1058_1x2032 -> New Battery:BAT_BH32T-C-G
- turned BT1 to -90 degrees
Connections:
- D1 pad 1: Net-(BT1--) -> Net-(D1-K)
- SW1 pad 1: Net-(BT1-+) -> Net-(BT1-Pad+)
Routing:
- net Net-(BT1--): track 68.7 -> 0.00 mm
- net Net-(D1-K): track 0.00 -> 50.1 mm
- net Net-(BT1-Pad+): track 0.00 -> 44.2 mm
- net Net-(BT1-+): track 14.5 -> 0.00 mm
