File: traffic_light/traffic_light.kicad_sch (KiCad schematic)
At the start: 7 parts, among them J1 Conn_01x04_Pin

Commit message: holes and trackes
Changed lines of the file:
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@@
 		(dnp no)
 		(property "Reference" "R1"
-			(at 107.696 64.262 90)
+			(at 118.11 68.58 90)
 			(effects
 				(font
@@
 		)
 		(property "Value" "330"
-			(at 107.696 66.802 90)
+			(at 118.11 71.12 90)
 			(effects
 				(font
@@
 		(dnp no)
 		(property "Reference" "D2"
-			(at 147.574 78.74 0)
+			(at 138.43 81.026 0)
 			(effects
 				(font
@@
 		)
 		(property "Value" "LED"
-			(at 147.574 81.28 0)
-			(effects
-				(font
+			(at 138.43 83.566 0)
+			(effects
+				(font
