File: traffic_light/traffic_light.kicad_pcb (KiCad board)
At the start: 2 copper layers, 32.6 x 22.6 mm, 7 parts, among them J1 Conn_01x04_Pin

Commit message: traffic light
Routing:
- net /GND: track 46.8 -> 0.00 mm
- added copper zone on B.Cu, net /GND
Other:
- board text added: "Eng.Ahmed Gamal 01286447720"
- board text added: "GND"
- board text added: "LED1"
- board text added: "LED2"
- board text added: "LED3"
- board text added: "Traffic Light V1"
Changed lines of the file:
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@@
 		(tags "Through hole angled pin header THT 1x04 2.00mm single row")
 		(property "Reference" "J1"
-			(at 1.97 -2.81 360)
+			(at 1.97 -2.81 0)
 			(layer "F.SilkS")
 			(effects
@@
 		)
 		(property "Value" "Conn_01x04_Pin"
-			(at 3.1 8 360)
+			(at 3.1 8 0)
 			(layer "F.Fab")
 			(effects
@@
 		)
 	)
+	(gr_rect
+		(start 113.99 57.7)
+		(end 120.14 60.07)
+		(stroke
+			(width 0.1)
+			(type default)
+		)
+		(fill none)
+		(layer "F.SilkS")
+	)
+	(gr_rect
+		(start 122.17 76.5)
+		(end 129.71 78.69)
+		(stroke
+			(width 0.1)
+			(type default)
+		)
+		(fill none)
+		(layer "F.SilkS")
+	)
 	(gr_circle
 		(center 102.7 58.2)
@@
 		(layer "Edge.Cuts")
 	)
-	(segment
-		(start 130.92 66.29)
-		(end 130.92 70.4)
-		(width 0.2)
-		(layer "B.Cu")
-		(net 1)
-	)
-	(segment
-		(start 106.63 60.57)
-		(end 126.76 60.57)
-		(width 0.2)
-		(layer "B.Cu")
-		(net 1)
-	)
-	(segment
-		(start 129.707789 60.625155)
-		(end 129.755155 60.625155)
-		(width 0.2)
-		(layer "B.Cu")
-		(net 1)
-	)
-	(segment
-		(start 129.652634 60.57)
-		(end 129.707789 60.625155)
-		(width 0.2)
-		(layer "B.Cu")
-		(net 1)
-	)
-	(segment
-		(start 129.47 71.85)
-		(end 129.13 71.85)
-		(width 0.2)
-		(layer "B.Cu")
-		(net 1)
-	)
-	(segment
-		(start 105.1 64.5)
-		(end 105.1 62.1)
-		(width 0.2)
-		(layer "B.Cu")
-		(net 1)
-	)
-	(segment
-		(start 130.92 70.4)
-		(end 129.47 71.85)
-		(width 0.2)
-		(layer "B.Cu")
-		(net 1)
-	)
-	(segment
-		(start 130.91 66.28)
-		(end 130.92 66.29)
-		(width 0.2)
-		(layer "B.Cu")
-		(net 1)
-	)
-	(segment
-		(start 105.1 62.1)
-		(end 106.63 60.57)
-		(width 0.2)
-		(layer "B.Cu")
-		(net 1)
-	)
-	(segment
-		(start 129.12 71.84)
-		(end 126.85 71.84)
-		(width 0.2)
-		(layer "B.Cu")
-		(net 1)
-	)
-	(segment
-		(start 129.13 71.85)
-		(end 129.12 71.84)
-		(width 0.2)
-		(layer "B.Cu")
-		(net 1)
-	)
-	(segment
-		(start 129.755155 60.625155)
-		(end 130.92 61.79)
-		(width 0.2)
-		(layer "B.Cu")
-		(net 1)
-	)
-	(segment
-		(start 126.76 60.57)
-		(end 129.652634 60.57)
-		(width 0.2)
-		(layer "B.Cu")
-		(net 1)
-	)
-	(segment
-		(start 130.92 61.79)
-		(end 130.92 66.29)
-		(width 0.2)
-		(layer "B.Cu")
-		(net 1)
-	)
-	(segment
-		(start 126.76 66.28)
-		(end 130.91 66.28)
-		(width 0.2)
-		(layer "B.Cu")
-		(net 1)
+	(gr_text "LED3"
+		(at 106.26 66.67 0)
+		(layer "F.SilkS")
+		(effects
+			(font
+				(size 0.5 0.5)
+				(thickness 0.1)
+			)
+			(justify left bottom)
+		)
+	)
+	(gr_text "LED2"
+		(at 106.34 68.68 0)
+		(layer "F.SilkS")
+		(effects
+			(font
+				(size 0.5 0.5)
+				(thickness 0.1)
+			)
+			(justify left bottom)
+		)
+	)
+	(gr_text "LED1"
+		(at 106.36 70.72 0)
+		(layer "F.SilkS")
+		(effects
+			(font
+				(size 0.5 0.5)
+				(thickness 0.1)
+			)
+			(justify left bottom)
+		)
+	)
+	(gr_text "Eng.Ahmed Gamal\n01286447720"
+		(at 122.51 78.31 0)
+		(layer "F.SilkS")
+		(effects
+			(font
+				(size 0.5 0.5)
+				(thickness 0.125)
+				(bold yes)
+				(italic yes)
+			)
+			(justify left bottom)
+		)
+	)
+	(gr_text "Traffic Light\nV1"
+		(at 116.97 59.77 0)
+		(layer "F.SilkS")
+		(effects
+			(font
+				(size 0.6 0.6)
+				(thickness 0.1)
+			)
+			(justify bottom)
+		)
+	)
+	(gr_text "GND"
+		(at 106.41 65.07 0)
+		(layer "F.SilkS")
+		(effects
+			(font
+				(size 0.5 0.5)
+				(thickness 0.1)
+			)
+			(justify left bottom)
+		)
 	)
 	(segment
@@
 		(net 7)
 	)
+	(zone
+		(net 1)
+		(net_name "/GND")
+		(layer "B.Cu")
+		(hatch edge 0.5)
+		(connect_pads
+			(clearance 0.5)
+		)
+		(min_thickness 0.25)
+		(filled_areas_thickness no)
+		(fill yes
+			(thermal_gap 0.5)
+			(thermal_bridge_width 0.5)
+		)
+		(polygon
+			(pts
+				(xy 100.98 56.7) (xy 133.52 56.71) (xy 133.52 79.3) (xy 100.95 79.3)
+			)
+		)
+	)
 )
