File: DC_DC_Power_Supply_5V_3.3V/DC_DC_Power_Supply_5V_3.3V.kicad_pcb (KiCad board)
At the start: 2 copper layers, 52.1 x 24.7 mm, 8 parts, among them J1 Screw_Terminal_01x02, J2 USB_B_Micro, U2 AMS1117CD-3.3

Commit message: DC_DC Power Supply
Other:
- board text added: "5v to 3.3v"
- board text added: "Simple Voltage Regulator"
- board text removed: "Eng.Ahmed Gamal V1.0"
Changed lines of the file:
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@@
 			(outputformat 1)
 			(mirror no)
-			(drillshape 1)
+			(drillshape 0)
 			(scaleselection 1)
-			(outputdirectory "")
+			(outputdirectory "gerbers/")
 		)
 	)
@@
 		(layer "Edge.Cuts")
 	)
-	(gr_text "Eng.Ahmed Gamal\nV1.0"
-		(at 112.22 146.17 0)
+	(gr_text "5v to 3.3v"
+		(at 115.66 146.21 0)
 		(layer "F.SilkS")
 		(effects
@@
 				(thickness 0.1)
 			)
-			(justify left bottom)
+			(justify bottom)
 		)
 	)
+	(gr_text "Simple Voltage Regulator\n"
+		(at 116.71 144.62 0)
+		(layer "F.SilkS" knockout)
+		(effects
+			(font
+				(size 1 1)
+				(thickness 0.16)
+				(bold yes)
+			)
+			(justify bottom)
+		)
+	)
