File: Battery_Charger/Battery_Charger.kicad_sch (KiCad schematic)
At the start: 2 parts, among them J1 USB_B_Micro, U2 MCP73831-2-OT

Commit message: Battery Charger
Parts:
- added C2, C3: C_Polarized, Capacitor_SMD:C_1206_3216Metric, symbol Device:C_Polarized
- added D1: LED, LED_SMD:LED_1206_3216Metric, symbol Device:LED
- added J2: Conn_01x02_Socket, Connector_JST:JST_PH_S2B-PH-K_1x02_P2.00mm_Horizontal, symbol Connector:Conn_01x02_Socket
- added R1, R2: R, Resistor_SMD:R_1206_3216Metric, symbol Device:R
- J1: footprint (none) -> Connector_USB:USB_Micro-B_Molex_47346-0001
Connections:
- net LED_STAT: now reaches U2.1 (STAT)
- net LED_STAT: now also D1.1 (K)
- net GND: now reaches U2.2 (V_{SS})
- net GND: now also J1.5 (GND), J1.6 (Shield), C2.2, C3.2, J2.2 (Pin_2), R1.1
- net V_BAT: now reaches U2.3 (V_{BAT})
- net V_BAT: now also C2.1, J2.1 (Pin_1)
- net VCC: now reaches U2.4 (V_{DD})
- net VCC: now also J1.1 (VBUS), C3.1, R2.2
- net at U2.5 (PROG): now also R1.2
- new net: D1.2 (A), R2.1
- no-connect marks 0 -> 3
Other:
- moved on the sheet: J1
