File: IR_Sensor_Circuit/IR_Sensor_Circuit.kicad_sch (KiCad schematic)
At the start: 9 parts, among them J1 Conn_01x03_Pin, U1 LM358

Commit message: IR Circuit
Parts:
- removed R4: R, symbol Device:R
Changed lines of the file:
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@@
-	)
-	(symbol
-		(lib_id "Device:R")
-		(at 189.23 124.46 0)
-		(unit 1)
-		(exclude_from_sim no)
-		(in_bom yes)
-		(on_board yes)
-		(dnp no)
-		(fields_autoplaced yes)
-		(property "Reference" "R4"
-			(at 191.77 123.1899 0)
-			(effects
-				(font
-					(size 1.27 1.27)
-				)
-				(justify left)
-			)
-		)
-		(property "Value" "R"
-			(at 191.77 125.7299 0)
-			(effects
-				(font
-					(size 1.27 1.27)
-				)
-				(justify left)
-			)
-		)
-		(property "Footprint" ""
-			(at 187.452 124.46 90)
-			(effects
-				(font
-					(size 1.27 1.27)
-				)
-				(hide yes)
-			)
-		)
-		(property "Datasheet" "~"
-			(at 189.23 124.46 0)
-			(effects
-				(font
-					(size 1.27 1.27)
-				)
-				(hide yes)
-			)
-		)
-		(property "Description" "Resistor"
-			(at 189.23 124.46 0)
-			(effects
-				(font
-					(size 1.27 1.27)
-				)
-				(hide yes)
-			)
-		)
-		(pin "1"
-		)
-		(pin "2"
-		)
-		(instances
-			(project "IR_Sensor_Circuit"
-				(path "/70757889-7f82-480f-8e64-5199b01bf6a8"
-					(reference "R4")
-					(unit 1)
-				)
-			)
-		)
 	)
 	(symbol

Commit message: IR Circuit
Parts:
- added R2: 10K, Resistor_SMD:R_1206_3216Metric, symbol Device:R
- added unit 2 of U1
- added unit 3 of U1
- D1: value LED -> IR_LED; footprint (none) -> LED_SMD:LED_1206_3216Metric
- D2: value LED -> PhotoDiod_LED; footprint (none) -> LED_SMD:LED_1206_3216Metric
- D3: footprint (none) -> LED_SMD:LED_1206_3216Metric
- J1: footprint (none) -> Connector_PinHeader_2.54mm:PinHeader_1x03_P2.54mm_Horizontal
- R1: value R -> 100; footprint (none) -> Resistor_SMD:R_1206_3216Metric
- R3: footprint (none) -> Resistor_SMD:R_1206_3216Metric
- RV1: value R_Potentiometer -> 10K_R_Potentiometer; footprint (none) -> Potentiometer_SMD:Potentiometer_Bourns_3314J_Vertical
- U1: footprint (none) -> Package_TO_SOT_SMD:SOT-23-8
Connections:
- net GND: now also R2.2, U1.4 (V-)
- net VCC: now also RV1.1, U1.8 (V+)
- net POT_V: now reaches RV1.2, U1.2 (-)
- net at D1.1 (K), R1.1: no longer U1.3 (+)
- net PHD_V: now reaches D2.2 (A)
- net PHD_V: now also U1.3 (+), R2.1; no longer RV1.1
- no-connect marks 0 -> 3
Other:
- moved on the sheet: R1

Commit message: IR Circuit
Connections:
- net OUTPUT: now also J1.1 (Pin_1); no longer J1.3 (Pin_3)
- net VCC: now also J1.3 (Pin_3); no longer J1.1 (Pin_1)
Changed lines of the file:
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@@
 	(wire
 		(pts
-			(xy 43.18 73.66) (xy 57.15 73.66)
+			(xy 43.18 73.66) (xy 48.26 73.66)
 		)
 		(stroke
@@
 	(wire
 		(pts
-			(xy 57.15 54.61) (xy 57.15 73.66)
-		)
-		(stroke
-			(width 0)
-			(type default)
-		)
-	)
-	(wire
-		(pts
 			(xy 127 67.31) (xy 127 54.61)
 		)
@@
 	(wire
 		(pts
+			(xy 43.18 76.2) (xy 48.26 76.2)
+		)
+		(stroke
+			(width 0)
+			(type default)
+		)
+	)
+	(wire
+		(pts
 			(xy 81.28 90.17) (xy 97.79 90.17)
 		)
@@
 	(wire
 		(pts
-			(xy 43.18 76.2) (xy 57.15 76.2)
-		)
-		(stroke
-			(width 0)
-			(type default)
-		)
-	)
-	(wire
-		(pts
-			(xy 57.15 76.2) (xy 57.15 90.17)
-		)
-		(stroke
-			(width 0)
-			(type default)
-		)
-	)
-	(wire
-		(pts
 			(xy 121.92 81.28) (xy 114.3 81.28)
 		)
@@
 		)
 	)
-	(label "OUTPUT"
-		(at 48.26 78.74 0)
+	(label "GND"
+		(at 57.15 90.17 0)
 		(fields_autoplaced yes)
 		(effects
@@
 	)
 	(label "VCC"
-		(at 48.26 73.66 0)
+		(at 48.26 78.74 0)
 		(fields_autoplaced yes)
 		(effects
@@
 		(fields_autoplaced yes)
 		(effects
+			(font
+				(size 1.27 1.27)
+			)
+			(justify left bottom)
+		)
+	)
+	(label "VCC"
+		(at 57.15 54.61 0)
+		(fields_autoplaced yes)
+		(effects
+			(font
+				(size 1.27 1.27)
+			)
+			(justify left bottom)
+		)
+	)
+	(label "OUTPUT"
+		(at 48.26 73.66 0)
+		(fields_autoplaced yes)
+		(effects

Commit message: IR Sensor
Parts:
- D1: footprint LED_SMD:LED_1206_3216Metric -> LED_THT:LED_D5.0mm_Horizontal_O1.27mm_Z3.0mm_IRBlack
- D2: footprint LED_SMD:LED_1206_3216Metric -> LED_THT:LED_D5.0mm_Horizontal_O1.27mm_Z3.0mm_IRGrey
Changed lines of the file:
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@@
 			)
 		)
-		(property "Footprint" "LED_SMD:LED_1206_3216Metric"
+		(property "Footprint" "LED_THT:LED_D5.0mm_Horizontal_O1.27mm_Z3.0mm_IRGrey"
 			(at 97.79 60.96 0)
 			(effects
@@
 			)
 		)
-		(property "Footprint" "LED_SMD:LED_1206_3216Metric"
+		(property "Footprint" "LED_THT:LED_D5.0mm_Horizontal_O1.27mm_Z3.0mm_IRBlack"
 			(at 81.28 60.96 0)
 			(effects
