File: IR_Sensor_Circuit/IR_Sensor_Circuit.kicad_pcb (KiCad board)
At the start: 2 copper layers, 9 parts, among them J1 Conn_01x03_Pin, U1 LM358

Commit message: IR Circuit
Parts:
- moved J1 126.4 mm to (59.9, 114.9), turned to 180 degrees
- moved R3 117.9 mm to (68.9, 121.4), turned to 180 degrees
- moved R1 113.9 mm to (70.7, 110.7), turned to -90 degrees
- moved U1 111.2 mm to (88.1, 107.9)
- moved D3 110.2 mm to (68.7, 116.0), turned to 180 degrees
- moved D1 106.2 mm to (70.6, 105.3), turned to 90 degrees
- moved R2 104.9 mm to (79.6, 110.4), turned to -90 degrees
- moved D2 97.3 mm to (79.4, 105.1), turned to -90 degrees
- moved RV1 96.0 mm to (96.6, 107.7), turned to -90 degrees
Connections:
- J1 pad 1: /VCC -> /OUTPUT
- J1 pad 3: /OUTPUT -> /VCC
Routing:
- net /VCC: track 0.00 -> 63.6 mm
- net Net-(R3-Pad1): track 0.00 -> 34.1 mm
- net /GND: track 0.00 -> 19.4 mm
- net /OUTPUT: track 0.00 -> 13.3 mm
- net /POT_V: track 0.00 -> 11.6 mm
- net /PHD_V: track 0.00 -> 10.1 mm
- net Net-(D1-K): track 0.00 -> 2.54 mm
- added copper zone on F.Cu, net /GND
Other:
- board outline added: 47.6 x 26.9 mm

Commit message: IR Sensor
Parts:
- D1: footprint LED_SMD:LED_1206_3216Metric -> LED_THT:LED_D5.0mm_Horizontal_O1.27mm_Z3.0mm_IRBlack
- D2: footprint LED_SMD:LED_1206_3216Metric -> LED_THT:LED_D5.0mm_Horizontal_O1.27mm_Z3.0mm_IRGrey
- moved D1 52.3 mm to (121.8, 115.8)
- moved D2 46.8 mm to (121.8, 124.9), turned to 90 degrees
- moved R1 41.1 mm to (111.3, 116.4)
- moved D3 37.4 mm to (105.5, 122.6), turned to -90 degrees
- moved R3 36.9 mm to (105.5, 116.1), turned to 90 degrees
- moved R2 34.1 mm to (111.4, 122.6), turned to 90 degrees
- moved J1 31.1 mm to (90.2, 121.6)
- moved RV1 17.4 mm to (98.5, 125.0), turned to 90 degrees
- moved U1 11.6 mm to (96.7, 115.7), turned to 90 degrees
Routing:
- net /OUTPUT: track 13.3 -> 59.7 mm
- net Net-(R3-Pad1): track 34.1 -> 0.00 mm
- net /GND: track 19.4 -> 0.00 mm
- net /POT_V: track 11.6 -> 0.00 mm
- net /VCC: track 63.6 -> 74.9 mm
- net Net-(D1-K): track 2.54 -> 11.2 mm
- net /PHD_V: track 10.1 -> 11.1 mm
- removed copper zone on F.Cu, net /GND
Other:
- board size 47.6 x 26.9 mm -> 39.5 x 25 mm

Commit message: STM32 UART
Parts:
- turned RV1 to -90 degrees
- turned U1 to -90 degrees
Routing:
- net /POT_V: track 0.00 -> 29.8 mm
- net /PHD_V: track 11.1 -> 32.7 mm, vias 0 -> 1
- net (no net): track 0.00 -> 13.8 mm, vias 0 -> 4
- net Net-(R3-Pad1): track 0.00 -> 13.3 mm
- net /VCC: track 74.9 -> 67.8 mm
- net /GND: track 0.00 -> 3.49 mm, vias 0 -> 2
- added copper zone on F.Cu, net /GND
