File: Assignment_1_Power_Supply/Assignment_1_Power_Supply.kicad_sch (KiCad schematic)
At the start: 12 parts, among them J1 Conn_01x02_Pin, J2 Conn_01x03_Pin, SW1 SW_Push_DPDT, T1 Transformer_1P_1S, U1 L7805, U2 AMS1117CD-3.3

Commit message: Ass1 Power Supply
Parts:
- C1, C2, C3, C4, C5: footprint (none) -> Capacitor_SMD:CP_Elec_8x5.4
- J1: footprint (none) -> Connector_PinHeader_2.54mm:PinHeader_1x02_P2.54mm_Vertical
- J2: footprint (none) -> Connector_PinHeader_2.54mm:PinHeader_1x03_P2.54mm_Vertical_SMD_Pin1Right
- SW1: footprint (none) -> Button_Switch_SMD:SW_DPDT_CK_JS202011JCQN
- T1: footprint (none) -> Transformer_THT:Transformer_NF_ETAL_P1165
- U1: footprint (none) -> Package_TO_SOT_SMD:TO-263-3_TabPin2
Connections:
- net 220/12 vAC: now reaches J1.1 (Pin_1), SW1.2 (B)
Changed lines of the file:
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@@
+	)
+	(junction
+		(at 35.56 77.47)
+		(diameter 0)
+		(color 0 0 0 0)
 	)
 	(junction
@@
 	(wire
 		(pts
+			(xy 35.56 77.47) (xy 39.37 77.47)
+		)
+		(stroke
+			(width 0)
+			(type default)
+		)
+	)
+	(wire
+		(pts
 			(xy 142.24 88.9) (xy 167.64 88.9)
 		)
@@
 	(wire
 		(pts
-			(xy 31.75 77.47) (xy 39.37 77.47)
+			(xy 31.75 77.47) (xy 35.56 77.47)
 		)
 		(stroke
@@
 		(pts
 			(xy 240.03 85.09) (xy 240.03 88.9)
+		)
+		(stroke
+			(width 0)
+			(type default)
+		)
+	)
+	(wire
+		(pts
+			(xy 35.56 64.77) (xy 35.56 77.47)
 		)
 		(stroke
@@
 	(label "12vAC"
 		(at 100.33 72.39 0)
+		(fields_autoplaced yes)
+		(effects
+			(font
+				(size 1.27 1.27)
+			)
+			(justify left bottom)
+		)
+	)
+	(label "220{slash}12 vAC"
+		(at 35.56 64.77 0)
 		(fields_autoplaced yes)
 		(effects
@@
 			)
 		)
-		(property "Footprint" ""
+		(property "Footprint" "Connector_PinHeader_2.54mm:PinHeader_1x03_P2.54mm_Vertical_SMD_Pin1Right"
 			(at 266.7 104.14 0)
 			(effects
@@
 			)
 		)
-		(property "Footprint" ""
+		(property "Footprint" "Capacitor_SMD:CP_Elec_8x5.4"
 			(at 261.3152 85.09 0)
 			(effects
@@
 			)
 		)
-		(property "Footprint" ""
+		(property "Footprint" "Connector_PinHeader_2.54mm:PinHeader_1x02_P2.54mm_Vertical"
 			(at 26.67 77.47 0)
 			(effects
@@
 			)
 		)
-		(property "Footprint" ""
+		(property "Footprint" "Package_TO_SOT_SMD:TO-263-3_TabPin2"
 			(at 168.275 81.28 0)
 			(effects
@@
 			)
 		)
-		(property "Footprint" ""
+		(property "Footprint" "Button_Switch_SMD:SW_DPDT_CK_JS202011JCQN"
 			(at 50.8 74.93 0)
 			(effects
@@
 			)
 		)
-		(property "Footprint" ""
+		(property "Footprint" "Capacitor_SMD:CP_Elec_8x5.4"
 			(at 201.6252 85.09 0)
 			(effects
@@
 			)
 		)
-		(property "Footprint" ""
+		(property "Footprint" "Capacitor_SMD:CP_Elec_8x5.4"
 			(at 143.2052 85.09 0)
 			(effects
@@
 			)
 		)
-		(property "Footprint" ""
+		(property "Footprint" "Transformer_THT:Transformer_NF_ETAL_P1165"
 			(at 85.09 77.47 0)
 			(effects
@@
 			)
 		)
-		(property "Footprint" ""
+		(property "Footprint" "Capacitor_SMD:CP_Elec_8x5.4"
 			(at 240.9952 85.09 0)
 			(effects
@@
 			)
 		)
-		(property "Footprint" ""
+		(property "Footprint" "Capacitor_SMD:CP_Elec_8x5.4"
 			(at 182.5752 85.09 0)
 			(effects
