File: Assignment_1_Power_Supply/Assignment_1_Power_Supply.kicad_pcb (KiCad board)
At the start: 2 copper layers, 44.2 x 65.6 mm, 12 parts, among them J1 Conn_01x02_Pin, J2 Conn_01x03_Pin, SW1 SW_Push_DPDT, T1 Transformer_1P_1S, U1 L7805, U2 AMS1117CD-3.3

Commit message: Ass1
Parts:
- moved J1 16.0 mm to (68.9, 98.6), turned to 90 degrees
- moved SW1 6.97 mm to (62.4, 103.2)
- moved T1 0.70 mm to (89.9, 101.2)
Routing:
- net /5v_OUTPUT: track 0.00 -> 120.6 mm
- net /12vDC: track 0.00 -> 50.7 mm
- net /GND_220vAC: track 20.0 -> 63.5 mm
- net /3v3_OUTPUT: track 0.00 -> 37.0 mm
- net /GND_AC: track 10.4 -> 28.4 mm
- net /220vAC: track 22.3 -> 32.6 mm
- net /GND: track 0.00 -> 7.87 mm
- net /12vAC: track 23.7 -> 31.2 mm
- net /220/12 vAC: track 15.6 -> 17.5 mm
- added copper zone on F.Cu, net /GND
Other:
- board text added: "220/12 VAC Input"
- board text added: "5,3.3 VDC Output"
- board text added: "Ahmed Gamal Ass 1 5 and 3.3 VDC PowerSupply imt School"

Commit message: Ass1
Parts:
- moved C2 1.32 mm to (84.8, 154.4)
Routing:
- net /3v3_OUTPUT: track 37.0 -> 43.2 mm
Other:
- board size 44.2 x 65.6 mm -> 44.2 x 66.4 mm
Changed lines of the file:
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@@
 			(outputformat 1)
 			(mirror no)
-			(drillshape 1)
+			(drillshape 0)
 			(scaleselection 1)
-			(outputdirectory "")
+			(outputdirectory "./")
 		)
 	)
@@
 	(footprint "Capacitor_SMD:CP_Elec_8x5.4"
 		(layer "F.Cu")
-		(at 83.81 155.29 90)
+		(at 84.77 154.38 90)
 		(descr "SMD capacitor, aluminum electrolytic, Nichicon, 8.0x5.4mm")
 		(tags "capacitor electrolytic")
@@
 		)
 		(fp_text user "${REFERENCE}"
-			(at 0 1.27 360)
+			(at 0 1.27 0)
 			(layer "F.Fab")
 			(effects
@@
 	(gr_rect
 		(start 52.32 95.19)
-		(end 96.49 160.8)
+		(end 96.49 161.64)
 		(stroke
 			(width 0.05)
@@
 	(segment
 		(start 68.47 158.085)
-		(end 70.485 160.1)
+		(end 70.385 160)
 		(width 0.2)
 		(layer "F.Cu")
@@
 	)
 	(segment
-		(start 82.34 159.84)
-		(end 82.34 159.81)
+		(start 58.9475 154.32)
+		(end 58.9475 148.02)
 		(width 0.2)
 		(layer "F.Cu")
@@
 	)
 	(segment
-		(start 70.485 160.1)
-		(end 82.08 160.1)
+		(start 70.385 160)
+		(end 82.15 160)
 		(width 0.2)
 		(layer "F.Cu")
@@
 	)
 	(segment
-		(start 82.34 159.81)
+		(start 82.15 160)
 		(end 83.81 158.34)
 		(width 0.2)
@@
 	)
 	(segment
-		(start 82.08 160.1)
-		(end 82.34 159.84)
-		(width 0.2)
-		(layer "F.Cu")
-		(net 3)
-	)
-	(segment
 		(start 62.725 155.995)
 		(end 60.4725 155.995)
@@
 		(polygon
 			(pts
-				(xy 52.33 95.19) (xy 96.48 95.19) (xy 96.48 160.8) (xy 52.33 160.8)
+				(xy 52.33 95.19) (xy 96.48 95.19) (xy 96.81 162.26) (xy 51.82 162.31)
 			)
 		)
@@
 		(polygon
 			(pts
-				(xy 52.33 95.19) (xy 96.48 95.19) (xy 96.48 160.81) (xy 52.33 160.8)
+				(xy 52.33 95.19) (xy 96.48 95.19) (xy 96.75 162.52) (xy 51.76 162.42)
 			)
 		)
