File: Atmega328p_MCU_DataLogger_board/Atmega328p_MCU_DataLogger_board.kicad_sch (KiCad schematic)
At the start: 16 parts, among them U1 24LC1025, U2 24LC1025, U3 ATMEGA328P-AU, U4 ds1337s+, Y1 Crystal, Y2 32.768 kHz

Commit message: MCU DataLogger
Parts:
- added BT1: Battery_Cell, symbol Device:Battery_Cell
- added C4: 0.1uF, symbol Device:C
- added C5: C, symbol Device:C
- added D1, D2: LED, symbol Device:LED
- added R8, R9: R, symbol Device:R
- R5: value R -> 10k
Connections:
- net GND: now also R6.2, U1.1 (A0), U1.2 (A1), U1.3 (A2), U1.4 (GND), U1.7 (WP), U2.4 (GND), U2.7 (WP), U3.21 (GND), U3.3 (GND), U3.5 (GND), BT1.2 (-), C4.2, C5.2, R8.2
- net SCK: now also R7.2, U1.6 (SCL), U2.6 (SCL), U3.17 (PB5(SCK/PCINT5)), D1.2 (A)
- net SDA: now also U1.5 (SDA), U2.5 (SDA), R9.2
- net VCC: now also R5.2, R7.1, U1.8 (VCC), U2.1 (A0), U2.2 (A1), U2.3 (A2), U2.8 (VCC), U3.18 (AVCC), U3.4 (VCC), U3.6 (VCC), BT1.1 (+), C5.1, D2.2 (A), R9.1
- net RESET: now reaches R5.1
- net RESET: now also U3.29 (PC6(*RESET/PCINT14))
- net at R6.1: now also D2.1 (K)
- net D3: now reaches U3.1 (PD3(PCINT19/OC2B/INT1))
- net D6: now reaches U3.10 (PD6(PCINT22/OC0A/AIN0))
- net D7: now reaches U3.11 (PD7(PCINT23/AIN1))
- net D8: now reaches U3.12 (PB0(PCINT0/CLKO/ICP1))
- net MOSI: now reaches U3.15 (PB3(PCINT3/OC2A/MOSI))
- net MISO: now reaches U3.16 (PB4(PCINT4/MISO))
- net D4: now reaches U3.2 (PD4(PCINT20/XCK/T0))
- net at U3.20 (AREF): now also C4.1
- net RX: now reaches U3.30 (PD0(RXD/PCINT16))
- net TX: now reaches U3.31 (PD1(TXD/PCINT17))
- net D2: now reaches U3.32 (PD2(INT0/PCINT18))
- net D5: now reaches U3.9 (PD5(PCINT21/OC0B/T1))
- new net: D1.1 (K), R8.1
- no-connect marks 0 -> 8
Other:
- title: (none) -> MCU DataLogger
- moved on the sheet: R5, R6, R7, U1, U2, Y1

Commit message: Project
Other:
- added sheet Connectors (untitled.kicad_sch)
- moved on the sheet: R7, R9, U1, U2

Commit message: Data Logger
Connections:
- net GND: no longer U3.3 (GND), U3.5 (GND)
- no-connect marks 8 -> 10
Other:
- sheet Connectors ports: added none; removed D2, D3, D4, D5, D6, D7, D8, GND, MISO, MOSI, RESET, RX, SCK, SDA, TX, VCC
- moved on the sheet: C2, C3, D1, R5, Y1

Commit message: Project
Parts:
- BT1: footprint (none) -> Connector_PinHeader_2.54mm:PinHeader_2x01_P2.54mm_Vertical
- C1, C2, C3, C4, C5: footprint (none) -> Capacitor_SMD:C_0805_2012Metric
- D1, D2: footprint (none) -> LED_SMD:LED_1206_3216Metric_Pad1.42x1.75mm_HandSolder
- R1, R2, R3, R4, R5, R6, R7, R8, R9: footprint (none) -> Resistor_SMD:R_1210_3225Metric
- U1, U2: footprint (none) -> Package_TO_SOT_SMD:SOT-223-8
- U3: footprint TQFP32_32A_MCH -> atmega328:TQFP32_32A_MCH
- U4: footprint 21-0041B_8_MXM -> DS1337s_RTC_RealTimeClock:21-0041B_8_MXM
- Y1, Y2: footprint (none) -> Crystal:Crystal_SMD_5032-2Pin_5.0x3.2mm
Changed lines of the file:
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@@
 			)
 		)
-		(property "Footprint" ""
+		(property "Footprint" "Resistor_SMD:R_1210_3225Metric"
 			(at 261.112 118.11 90)
 			(effects
@@
 			)
 		)
-		(property "Footprint" ""
+		(property "Footprint" "Resistor_SMD:R_1210_3225Metric"
 			(at 98.552 121.92 90)
 			(effects
@@
 			)
 		)
-		(property "Footprint" ""
+		(property "Footprint" "Resistor_SMD:R_1210_3225Metric"
 			(at 165.862 111.76 90)
 			(effects
@@
 			)
 		)
-		(property "Footprint" ""
+		(property "Footprint" "Resistor_SMD:R_1210_3225Metric"
 			(at 191.77 47.498 90)
 			(effects
@@
 			)
 		)
-		(property "Footprint" ""
+		(property "Footprint" "Resistor_SMD:R_1210_3225Metric"
 			(at 217.932 57.15 90)
 			(effects
@@
 			)
 		)
-		(property "Footprint" ""
+		(property "Footprint" "Capacitor_SMD:C_0805_2012Metric"
 			(at 234.6452 46.99 0)
 			(effects
@@
 			)
 		)
-		(property "Footprint" ""
+		(property "Footprint" "Resistor_SMD:R_1210_3225Metric"
 			(at 243.332 118.11 90)
 			(effects
@@
 			)
 		)
-		(property "Footprint" ""
+		(property "Footprint" "Connector_PinHeader_2.54mm:PinHeader_2x01_P2.54mm_Vertical"
 			(at 248.92 42.926 90)
 			(effects
@@
 			)
 		)
-		(property "Footprint" "TQFP32_32A_MCH"
+		(property "Footprint" "atmega328:TQFP32_32A_MCH"
 			(at 44.45 38.1 0)
 			(effects
@@
 			)
 		)
-		(property "Footprint" ""
+		(property "Footprint" "LED_SMD:LED_1206_3216Metric_Pad1.42x1.75mm_HandSolder"
 			(at 175.26 76.2 0)
 			(effects
@@
 			)
 		)
-		(property "Footprint" ""
+		(property "Footprint" "Resistor_SMD:R_1210_3225Metric"
 			(at 250.952 118.11 90)
 			(effects
@@
 			)
 		)
-		(property "Footprint" "21-0041B_8_MXM"
+		(property "Footprint" "DS1337s_RTC_RealTimeClock:21-0041B_8_MXM"
 			(at 170.18 119.38 0)
 			(effects
@@
 			)
 		)
-		(property "Footprint" ""
+		(property "Footprint" "Package_TO_SOT_SMD:SOT-223-8"
 			(at 73.66 124.46 0)
 			(effects
@@
 			)
 		)
-		(property "Footprint" ""
+		(property "Footprint" "Capacitor_SMD:C_0805_2012Metric"
 			(at 21.59 49.8348 0)
 			(effects
@@
 			)
 		)
-		(property "Footprint" ""
+		(property "Footprint" "Capacitor_SMD:C_0805_2012Metric"
 			(at 21.59 57.4548 0)
 			(effects
@@
 			)
 		)
-		(property "Footprint" ""
+		(property "Footprint" "Resistor_SMD:R_1210_3225Metric"
 			(at 104.902 121.92 90)
 			(effects
@@
 			)
 		)
-		(property "Footprint" ""
+		(property "Footprint" "Crystal:Crystal_SMD_5032-2Pin_5.0x3.2mm"
 			(at 24.13 54.61 0)
 			(effects
@@
 			)
 		)
-		(property "Footprint" ""
+		(property "Footprint" "Capacitor_SMD:C_0805_2012Metric"
 			(at 274.0152 121.92 0)
 			(effects
@@
 			)
 		)
-		(property "Footprint" ""
+		(property "Footprint" "LED_SMD:LED_1206_3216Metric_Pad1.42x1.75mm_HandSolder"
 			(at 219.71 43.18 0)
 			(effects
@@
 			)
 		)
-		(property "Footprint" ""
+		(property "Footprint" "Resistor_SMD:R_1210_3225Metric"
 			(at 177.292 80.01 90)
 			(effects
@@
 			)
 		)
-		(property "Footprint" ""
+		(property "Footprint" "Capacitor_SMD:C_0805_2012Metric"
 			(at 186.3852 76.2 0)
 			(effects
@@
 			)
 		)
-		(property "Footprint" ""
+		(property "Footprint" "Package_TO_SOT_SMD:SOT-223-8"
 			(at 38.1 123.19 0)
 			(effects
@@
 			)
 		)
-		(property "Footprint" ""
+		(property "Footprint" "Crystal:Crystal_SMD_5032-2Pin_5.0x3.2mm"
 			(at 152.4 120.65 0)
 			(effects
